File: co2-sensor.kicad_pcb (KiCad board)
At the start: 2 copper layers, 61 x 61 mm, 51 parts, among them J1 24-pin FPC Connector, J2 USB-C Receptacle, J3 JST 2-PH, Q1 AO3401A, Q2 AO3400A, SW1 SW_Push, SW2 SW_Push, SW3 SW_Push, SW4 SW_Push, SW5 SW_Push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

Commit message: More tweaking
Routing:
- net +BATT: track 59.6 -> 56.4 mm
- net Net-(D2-A): track 11.5 -> 10.6 mm
- net GND: track 98.5 -> 97.8 mm
- net /CO2_EN: vias 1 -> 2
- net /I2C_SDA: vias 8 -> 7
- net /CO2_NRDY: vias 1 -> 2
Changed lines of the file:
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@@
 		(sheetfile "co2-sensor.kicad_sch")
 		(attr smd)
-		(fp_line
-			(start -2.276988 -0.093828)
-			(end -2.276988 1.074879)
-			(stroke
-				(width 0.254)
-				(type solid)
-			)
-			(layer "F.SilkS")
-		)
-		(fp_line
-			(start -1.000076 -2.42507)
-			(end -1.000076 -1.225095)
-			(stroke
-				(width 0.254)
-				(type solid)
-			)
-			(layer "F.SilkS")
-		)
-		(fp_line
-			(start -1.000076 -2.42507)
-			(end 0.999924 -2.42507)
-			(stroke
-				(width 0.254)
-				(type solid)
-			)
-			(layer "F.SilkS")
-		)
-		(fp_line
-			(start -0.889078 1.074879)
-			(end -1.169012 1.074879)
-			(stroke
-				(width 0.254)
-				(type solid)
-			)
-			(layer "F.SilkS")
-		)
-		(fp_line
-			(start -0.889078 1.074879)
-			(end 0.888926 1.074879)
-			(stroke
-				(width 0.254)
-				(type solid)
-			)
-			(layer "F.SilkS")
-		)
-		(fp_line
-			(start 0.888926 1.074879)
-			(end 1.168707 1.074879)
-			(stroke
-				(width 0.254)
-				(type solid)
-			)
-			(layer "F.SilkS")
-		)
-		(fp_line
-			(start 0.999924 -2.42507)
-			(end 0.999924 -1.225095)
-			(stroke
-				(width 0.254)
-				(type solid)
-			)
-			(layer "F.SilkS")
-		)
-		(fp_line
-			(start 2.275006 -0.093828)
-			(end 2.275006 1.074879)
-			(stroke
-				(width 0.254)
-				(type solid)
-			)
-			(layer "F.SilkS")
-		)
 		(fp_circle
 			(center -2.279858 -2.552172)
@@
 		(sheetfile "co2-sensor.kicad_sch")
 		(attr smd)
-		(fp_line
-			(start -2.276988 -0.093828)
-			(end -2.276988 1.074879)
-			(stroke
-				(width 0.254)
-				(type solid)
-			)
-			(layer "F.SilkS")
-		)
-		(fp_line
-			(start -1.000076 -2.42507)
-			(end -1.000076 -1.225095)
-			(stroke
-				(width 0.254)
-				(type solid)
-			)
-			(layer "F.SilkS")
-		)
-		(fp_line
-			(start -1.000076 -2.42507)
-			(end 0.999924 -2.42507)
-			(stroke
-				(width 0.254)
-				(type solid)
-			)
-			(layer "F.SilkS")
-		)
-		(fp_line
-			(start -0.889078 1.074879)
-			(end -1.169012 1.074879)
-			(stroke
-				(width 0.254)
-				(type solid)
-			)
-			(layer "F.SilkS")
-		)
-		(fp_line
-			(start -0.889078 1.074879)
-			(end 0.888926 1.074879)
-			(stroke
-				(width 0.254)
-				(type solid)
-			)
-			(layer "F.SilkS")
-		)
-		(fp_line
-			(start 0.888926 1.074879)
-			(end 1.168707 1.074879)
-			(stroke
-				(width 0.254)
-				(type solid)
-			)
-			(layer "F.SilkS")
-		)
-		(fp_line
-			(start 0.999924 -2.42507)
-			(end 0.999924 -1.225095)
-			(stroke
-				(width 0.254)
-				(type solid)
-			)
-			(layer "F.SilkS")
-		)
-		(fp_line
-			(start 2.275006 -0.093828)
-			(end 2.275006 1.074879)
-			(stroke
-				(width 0.254)
-				(type solid)
-			)
-			(layer "F.SilkS")
-		)
 		(fp_circle
 			(center -2.279858 -2.552172)
@@
 	)
 	(segment
-		(start 159.385032 72.775924)
-		(end 159.385032 73.114968)
-		(width 0.2)
-		(layer "F.Cu")
-		(net 1)
-	)
-	(segment
 		(start 138.458549 119.3)
 		(end 139.234802 119.3)
@@
 	)
 	(segment
-		(start 145.857755 88.18551)
-		(end 146.18551 88.18551)
-		(width 0.2)
-		(layer "F.Cu")
-		(net 1)
-	)
-	(segment
 		(start 139.729622 98.010765)
 		(end 139.729622 97.510765)
@@
 	(segment
 		(start 131.401286 102)
-		(end 131.401286 86.401286)
+		(end 131.401286 84.681872)
 		(width 0.2)
 		(layer "F.Cu")
@@
 	)
 	(segment
-		(start 131.401286 84.681872)
-		(end 131.401286 86.401286)
-		(width 0.2)
-		(layer "F.Cu")
-		(net 7)
-	)
-	(segment
 		(start 146.683549 123.625)
 		(end 144.501071 121.442522)
@@
 	)
 	(segment
-		(start 159.438247 110.577687)
-		(end 158.738247 109.877687)
-		(width 0.2)
-		(layer "F.Cu")
-		(net 8)
-	)
-	(segment
 		(start 163.263247 111.127687)
 		(end 162.238247 111.127687)
@@
 	)
 	(segment
+		(start 161.099686 84.347448)
+		(end 186.147789 84.347448)
+		(width 0.2)
+		(layer "F.Cu")
+		(net 16)
+	)
+	(segment
+		(start 186.147789 84.347448)
+		(end 190.151074 80.344163)
+		(width 0.2)
+		(layer "F.Cu")
+		(net 16)
+	)
+	(segment
 		(start 134.007755 85.63551)
 		(end 135.918303 85.63551)
@@
 		(net 16)
 	)
+	(via
+		(at 161.099686 84.347448)
+		(size 0.6)
+		(drill 0.3)
+		(layers "F.Cu" "B.Cu")
+		(net 16)
+	)
 	(segment
-		(start 190.151074 80.344163)
-		(end 186.133074 84.362163)
+		(start 137.710554 84.362163)
+		(end 161.084971 84.362163)
 		(width 0.2)
 		(layer "B.Cu")
@@
 	)
 	(segment
-		(start 186.133074 84.362163)
-		(end 137.710554 84.362163)
+		(start 137.710554 84.362163)
+		(end 136.177755 85.894962)
 		(width 0.2)
 		(layer "B.Cu")
@@
 	)
 	(segment
-		(start 137.710554 84.362163)
-		(end 136.177755 85.894962)
+		(start 161.084971 84.362163)
+		(end 161.099686 84.347448)
 		(width 0.2)
 		(layer "B.Cu")
@@
 	)
 	(segment
+		(start 162.075837 85.424163)
+		(end 190.151074 85.424163)
+		(width 0.2)
+		(layer "F.Cu")
+		(net 20)
+	)
+	(segment
 		(start 135.538155 86.505779)
 		(end 136.793676 86.505779)
@@
 	)
 	(segment
+		(start 161 86.5)
+		(end 162.075837 85.424163)
+		(width 0.2)
+		(layer "F.Cu")
+		(net 20)
+	)
+	(segment
 		(start 135.302376 86.27)
 		(end 135.538155 86.505779)
@@
 		(net 20)
 	)
+	(via
+		(at 161 86.5)
+		(size 0.6)
+		(drill 0.3)
+		(layers "F.Cu" "B.Cu")
+		(net 20)
+	)
 	(segment
 		(start 139.023991 86.20248)
@@
 	)
 	(segment
-		(start 189.075237 86.5)
-		(end 190.151074 85.424163)
+		(start 159.245016 86.5)
+		(end 161 86.5)
 		(width 0.2)
 		(layer "B.Cu")
@@
 	)
 	(segment
-		(start 159.245016 86.5)
-		(end 189.075237 86.5)
-		(width 0.2)
-		(layer "B.Cu")
-		(net 20)
-	)
-	(segment
 		(start 137.150345 86.4)
 		(end 140.22016 86.4)
@@
 	)
 	(segment
-		(start 161.743247 117.772687)
-		(end 161.788247 117.817687)
-		(width 0.2)
-		(layer "F.Cu")
-		(net 23)
-	)
-	(segment
 		(start 146.437046 87.23551)
 		(end 147.082605 87.881069)
@@
 	)
 	(segment
-		(start 145.5 96)
-		(end 145.455542 96.044458)
-		(width 0.2)
-		(layer "F.Cu")
-		(net 36)
-	)
-	(segment
 		(start 141.044458 96.044458)
 		(end 145.455542 96.044458)
@@
 	)
 	(via
-		(at 141 97)
-		(size 0.6)
-		(drill 0.3)
-		(layers "F.Cu" "B.Cu")
-		(net 37)
-	)
-	(via
 		(at 137.252498 93.752498)
 		(size 0.6)
@@
 	)
 	(segment
-		(start 138.458549 122.75)
-		(end 138.43355 122.774999)
-		(width 0.2)
-		(layer "F.Cu")
-		(net 38)
-	)
-	(segment
 		(start 137.528548 122.75)
 		(end 137.503548 122.725)
@@
 	)
 	(segment
-		(start 138.458549 123.25)
-		(end 138.43355 123.225001)
-		(width 0.2)
-		(layer "F.Cu")
-		(net 39)
-	)
-	(segment
 		(start 135.225 119.453418)
 		(end 135.517678 119.16074)
@@
 	)
 	(segment
-		(start 163.926743 112.926743)
-		(end 163.957023 112.896463)
-		(width 0.2)
-		(layer "B.Cu")
-		(net 44)
-	)
-	(segment
 		(start 160.435512 116.417974)
 		(end 163.926743 112.926743)
@@
 	)
 	(segment
-		(start 161.243247 117.772687)
-		(end 161.288247 117.817687)
-		(width 0.2)
-		(layer "F.Cu")
-		(net 45)
-	)
-	(segment
 		(start 161.243247 119.072688)
 		(end 161.243247 117.772687)
@@
 	)
 	(segment
-		(start 142.342641 118.155345)
-		(end 139.025 114.837704)
+		(start 139.025 111.5)
+		(end 140.3375 111.5)
 		(width 0.2)
 		(layer "F.Cu")
@@
 	)
 	(segment
-		(start 139.025 111.5)
-		(end 140.3375 111.5)
+		(start 140.443857 100.5)
+		(end 141.95 100.5)
 		(width 0.2)
 		(layer "F.Cu")
@@
 	)
 	(segment
-		(start 140.443857 100.5)
-		(end 141.95 100.5)
+		(start 142.342641 118.155345)
+		(end 139.025 114.837704)
 		(width 0.2)
 		(layer "F.Cu")
@@
 	)
 	(segment
-		(start 139.025 114.837704)
-		(end 139.025 108.360219)
-		(width 0.2)
-		(layer "F.Cu")
-		(net 57)
-	)
-	(segment
 		(start 140.225 102.225)
 		(end 142.5 99.95)
@@
 		(width 0.2)
 		(layer "F.Cu")
+		(net 57)
+	)
+	(segment
+		(start 139.025 114.837704)
+		(end 139.025 111.5)
+		(width 0.2)
+		(layer "F.Cu")
